File: LedGateController.kicad_pcb (KiCad board)
At the start: 2 copper layers, 144.5 x 25 mm, 52 parts, among them J1 GPIO, J2 SWD, J3 LED_OUT, Q1 FS8205A, Q2 AO3400A, Q3 AO3401A, SW1 BUTTON, SW2 ON_OFF, U1 STM32F030F4Px, U2 MT3608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

Commit message: Change rev. text
Other:
- board text added: "WS28xx LED Driver Rev. 2 github.com/knifa"
- board text removed: "WS28xx LED Driver Rev. 1 github.com/knifa"
Changed lines of the file:
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@@
     (effects (font (size 1 1) (thickness 0.16)) (justify left mirror))
   )
-  (gr_text "WS28xx LED Driver\nRev. 1\ngithub.com/knifa" (at 66.25 32.5) (layer B.SilkS)
+  (gr_text "WS28xx LED Driver\nRev. 2\ngithub.com/knifa" (at 66.25 32.5) (layer B.SilkS)
     (effects (font (size 3 3) (thickness 0.6)) (justify mirror))
   )
