File: LedGateController.kicad_pcb (KiCad board)
At the start: 2 copper layers, 144.5 x 25 mm, 52 parts, among them J1 GPIO, J2 SWD, J3 LED_OUT, Q1 FS8205A, Q2 AO3400A, Q3 AO3401A, SW1 BUTTON, SW2 ON_OFF, U1 STM32F030F4Px, U2 MT3608, U3 DW01, U4 XC6206P332MR, U5 PI4ULS5V201

Commit message: Remove unneeded ground vias
Routing:
- net GND: vias 24 -> 22
Changed lines of the file:
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@@
     (thickness 1.6)
     (drawings 24)
-    (tracks 298)
+    (tracks 296)
     (zones 0)
     (modules 52)
@@
   (gr_line (start 20.5 23.25) (end 20.5 41.75) (layer Edge.Cuts) (width 0.05))
   (segment (start 101.675 27.575) (end 102.975 27.575) (width 2) (layer F.Cu) (net 1))
-  (segment (start 106.750001 22.149999) (end 107.5 21.4) (width 0.5) (layer F.Cu) (net 1))
-  (segment (start 101.675 27.575) (end 101.675 27.225) (width 0.5) (layer F.Cu) (net 1))
-  (segment (start 101.675 27.225) (end 106.750001 22.149999) (width 0.5) (layer F.Cu) (net 1))
   (segment (start 96.75 32.5) (end 101.675 27.575) (width 2) (layer F.Cu) (net 1))
   (segment (start 30.62 32.5) (end 96.75 32.5) (width 2) (layer F.Cu) (net 1))
+  (segment (start 101.675 27.225) (end 106.750001 22.149999) (width 0.5) (layer F.Cu) (net 1))
+  (segment (start 101.675 27.575) (end 101.675 27.225) (width 0.5) (layer F.Cu) (net 1))
+  (segment (start 106.750001 22.149999) (end 107.5 21.4) (width 0.5) (layer F.Cu) (net 1))
   (segment (start 107.13169 34.179189) (end 109.320811 34.179189) (width 0.75) (layer F.Cu) (net 2))
   (segment (start 107.13169 34.179189) (end 104.059189 34.179189) (width 0.75) (layer F.Cu) (net 2))
@@
   (via (at 145.625 41.2) (size 0.75) (drill 0.45) (layers F.Cu B.Cu) (net 4))
   (via (at 147.125 41.2) (size 0.75) (drill 0.45) (layers F.Cu B.Cu) (net 4))
-  (via (at 102.1 36.85) (size 0.75) (drill 0.45) (layers F.Cu B.Cu) (net 4))
-  (via (at 102.1 23.75) (size 0.75) (drill 0.45) (layers F.Cu B.Cu) (net 4))
   (via (at 131.8 29.875) (size 0.75) (drill 0.45) (layers F.Cu B.Cu) (net 4))
   (via (at 131.8 31.375) (size 0.75) (drill 0.45) (layers F.Cu B.Cu) (net 4))

Commit message: Update schematic
Parts:
- removed SW2: ON_OFF, SamacSys_Parts:SK12D07VG4NSPA
- added C15: 1u, Capacitor_SMD:C_0805_2012Metric, F.Cu at (96.8, -3.22)
- added C16: 100n, Capacitor_SMD:C_0805_2012Metric, F.Cu at (87.9, 3.43)
- added C17: 100n, Capacitor_SMD:C_0805_2012Metric, F.Cu at (92.4, -0.27)
- added C18: 4u7, Capacitor_SMD:C_0805_2012Metric, F.Cu at (100.9, -7.77)
- added C19: 4u7, Capacitor_SMD:C_0805_2012Metric, F.Cu at (87.9, 6.38)
- added D3: D_x2_KCom_AAK, Package_TO_SOT_SMD:SOT-23, F.Cu at (83.5, -0.32)
- added D4: D_x2_KCom_AAK, Package_TO_SOT_SMD:SOT-23, F.Cu at (92.0, -6.97)
- added D5: CHARGE_LED, LED_SMD:LED_0805_2012Metric, F.Cu at (83.5, 8.02)
- added J4: USB_B_Micro, SamacSys_Parts:U254051T4BHJ25S2S, F.Cu at (115.0, 23.5)
- added J5: TP4056, SamacSys_Parts:SOIC127P600X175-9N, F.Cu at (85.5, -5.92)
- added JP2: BOOT, Jumper:SolderJumper-2_P1.3mm_Open_Pad1.0x1.5mm, F.Cu at (123.4, -7.75)
- added Q4: AO3401A, Package_TO_SOT_SMD:SOT-23, F.Cu at (83.5, 4.23)
- added Q5: AO3400A, Package_TO_SOT_SMD:SOT-23, F.Cu at (87.9, -0.32)
- added Q6: AO3401A, Package_TO_SOT_SMD:SOT-23, F.Cu at (96.4, -6.97)
- added R11: 100K, Resistor_SMD:R_0805_2012Metric, F.Cu at (92.4, 2.68)
- added R12: 100K, Resistor_SMD:R_0805_2012Metric, F.Cu at (92.4, -3.22)
- added R13: 1K, Resistor_SMD:R_0805_2012Metric, F.Cu at (96.8, -0.27)
- added R14: 1K, Resistor_SMD:R_0805_2012Metric, F.Cu at (105.3, -7.77)
- added R15: 1K5, Resistor_SMD:R_0805_2012Metric, F.Cu at (92.3, 5.63)
- added R16: 100K, Resistor_SMD:R_0805_2012Metric, F.Cu at (101.2, -4.82)
- added R17: 100, Resistor_SMD:R_0805_2012Metric, F.Cu at (96.8, 2.68)
- added R18: 100K, Resistor_SMD:R_0805_2012Metric, F.Cu at (101.2, -1.87)
- added R19: 100K, Resistor_SMD:R_0805_2012Metric, F.Cu at (105.6, -4.82)
- added R20: 100K, Resistor_SMD:R_0805_2012Metric, F.Cu at (109.7, -7.77)
- added R21: 1.5K, Resistor_SMD:R_0805_2012Metric, F.Cu at (96.7, 5.63)
- added R22: 1.5K, Resistor_SMD:R_0805_2012Metric, F.Cu at (101.2, 1.08)
- added R23: 100K, Resistor_SMD:R_0805_2012Metric, F.Cu at (105.6, -1.87)
- added R24: 250, Resistor_SMD:R_0805_2012Metric, F.Cu at (110.0, -4.82)
- C1, C10, C11, C12, C14, C2, C3, C4, C5, C6, C8, C9: footprint Capacitor_SMD:C_0805_2012Metric_Pad1.15x1.40mm_HandSolder -> Capacitor_SMD:C_0805_2012Metric
- C7: value 1u -> 100n; footprint Capacitor_SMD:C_0805_2012Metric_Pad1.15x1.40mm_HandSolder -> Capacitor_SMD:C_0805_2012Metric
- D2: value LED -> PWR_LED; footprint LED_SMD:LED_0805_2012Metric_Pad1.12x1.40mm_HandSolder -> LED_SMD:LED_0805_2012Metric
- Q2: value AO3400A -> AO3401A
- R1, R3, R4, R5, R6, R9: footprint Resistor_SMD:R_0805_2012Metric_Pad1.15x1.40mm_HandSolder -> Resistor_SMD:R_0805_2012Metric
- R10: value 100K -> 150K; footprint Resistor_SMD:R_0805_2012Metric_Pad1.15x1.40mm_HandSolder -> Resistor_SMD:R_0805_2012Metric
- R2: value 100K -> 100; footprint Resistor_SMD:R_0805_2012Metric_Pad1.15x1.40mm_HandSolder -> Resistor_SMD:R_0805_2012Metric
- R7: value 100 -> 100K; footprint Resistor_SMD:R_0805_2012Metric_Pad1.15x1.40mm_HandSolder -> Resistor_SMD:R_0805_2012Metric
- R8: value 150 -> 250; footprint Resistor_SMD:R_0805_2012Metric_Pad1.15x1.40mm_HandSolder -> Resistor_SMD:R_0805_2012Metric
- TP7: value BATT_ADC -> BATT_SENSE
- U1: value STM32F030F4Px -> STM32F103C8Tx; footprint Package_SO:TSSOP-20_4.4x6.5mm_P0.65mm -> Package_QFP:LQFP-48_7x7mm_P0.5mm
- U2, U3, U5: footprint Package_TO_SOT_SMD:SOT-23-6_Handsoldering -> Package_TO_SOT_SMD:SOT-23-6
- moved R2 43.7 mm to (108.2, 9.25)
- moved R7 17.1 mm to (104.2, 9.25)
Connections:
- C10 pad 1: +5V -> Net-(C10-Pad1)
- C10 pad 2: GND -> Net-(C10-Pad2)
- C11 pad 2: GND -> Net-(C10-Pad2)
- C13 pad 1: +5V -> Net-(C13-Pad1)
- C13 pad 2: Net-(C13-Pad2) -> GND
- C2 pad 1: +BATT_SW -> /+BATT_SWITCH
- C3 pad 1: /NRST -> +3V3
- C7 pad 1: +3V3 -> GND
- C7 pad 2: GND -> /NRST
- J1 pad 3: /PA2 -> Net-(J1-Pad3)
- J1 pad 4: /PA1 -> Net-(J1-Pad4)
- J1 pad 5: /PA5 -> Net-(J1-Pad5)
- J1 pad 6: /PA6 -> Net-(J1-Pad6)
- J2 pad 5: /SWDCLK -> /SWCLK
- J3 pad 1: Net-(C13-Pad2) -> GND
- J3 pad 3: +5V -> Net-(C13-Pad1)
- L1 pad 1: +BATT_SW -> /+BATT_SWITCH
- Q2 pad 2: GND -> /+BATT_SWITCH
- Q2 pad 3: Net-(C13-Pad2) -> Net-(Q2-Pad3)
- Q3 pad 3: +BATT_SW -> /+BATT_SWITCH
- R10 pad 1: /BATT_ADC -> /BATT_SENSE
- R2 pad 1: Net-(R2-Pad1) -> Net-(Q2-Pad1)
- R2 pad 2: GND -> VBUS
- R6 pad 2: Net-(Q2-Pad1) -> Net-(Q4-Pad1)
- R7 pad 1: +BATT -> Net-(Q2-Pad1)
- R7 pad 2: Net-(R7-Pad2) -> GND
- R8 pad 1: +BATT_SW -> /+BATT_SWITCH
- R9 pad 1: +BATT_SW -> /+BATT_SWITCH
- R9 pad 2: /BATT_ADC -> /BATT_SENSE
- SW1 pad 2: GND -> +BATT
- TP7 pad 1: /BATT_ADC -> /BATT_SENSE
- U1 pad 1: Net-(R2-Pad1) -> Net-(U1-Pad1)
- U1 pad 10: /BATT_ADC -> Net-(U1-Pad10)
- U1 pad 11: /PA5 -> /LED_EN
- U1 pad 12: /PA6 -> /PWR_LATCH
- U1 pad 14: Net-(U1-Pad14) -> /BATT_SENSE
- U1 pad 15: GND -> Net-(U1-Pad15)
- U1 pad 16: +3V3 -> Net-(U1-Pad16)
- U1 pad 18: /LED_DATA_3V3 -> Net-(U1-Pad18)
- U1 pad 19: /SWDIO -> Net-(U1-Pad19)
- U1 pad 20: /SWDCLK -> Net-(U1-Pad20)
- U1 pad 4: /NRST -> Net-(U1-Pad4)
- U1 pad 5: +3V3 -> Net-(U1-Pad5)
- U1 pad 6: /LED_EN -> Net-(U1-Pad6)
- U1 pad 7: /PA1 -> /NRST
- U1 pad 8: /PA2 -> GND
- U1 pad 9: /BUTTON -> +3V3
- U2 pad 4: +BATT_SW -> Net-(Q2-Pad3)
- U2 pad 5: +BATT_SW -> /+BATT_SWITCH
- U4 pad 1: GND -> Net-(C10-Pad2)
- U4 pad 3: +5V -> Net-(C10-Pad1)
Routing:
- net +3V3: track 84.1 -> 25.9 mm, vias 5 -> 2
- net /LED_DATA_3V3: track 32.5 -> 3.55 mm, vias 1 -> 0
- net /SWDCLK: track 24.0 -> 0.00 mm, vias 1 -> 0
- net /SWDIO: track 22.9 -> 0.24 mm, vias 1 -> 0
- net /PA6: track 17.6 -> 0.00 mm, vias 1 -> 0
- net /PA5: track 17.4 -> 0.00 mm, vias 1 -> 0
- net /BUTTON: track 16.9 -> 0.00 mm, vias 1 -> 0
- net /+BATT_SWITCH: track 0.00 -> 16.9 mm
- net +BATT_SW: track 16.9 -> 0.00 mm
- net /BATT_ADC: track 15.0 -> 0.00 mm, vias 1 -> 0
- net /PA2: track 14.1 -> 0.00 mm, vias 1 -> 0
- net /LED_EN: track 13.9 -> 0.00 mm, vias 2 -> 0
- net /NRST: track 15.3 -> 1.62 mm, vias 1 -> 0
- net /PA1: track 13.1 -> 0.00 mm, vias 1 -> 0
- net Net-(C13-Pad2): track 12.9 -> 0.00 mm
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
Commit message: Rewire top section
Parts:
- TP1, TP2, TP3, TP4, TP5, TP6, TP7: footprint TestPoint:TestPoint_THTPad_D1.5mm_Drill0.7mm -> TestPoint:TestPoint_Pad_D1.0mm
- moved Q4 117.8 mm to (194.2, 44.6)
- moved R12 110.0 mm to (191.4, 44.7), turned to 90 degrees
- moved TP1 83.0 mm to (25.2, 32.5)
- moved TP2 82.6 mm to (25.2, 35.8), turned to 180 degrees
- moved J2 78.5 mm to (199.1, -36.5)
- moved R11 76.1 mm to (168.5, 4.60)
- moved C15 72.7 mm to (169.5, -1.40)
- moved R15 69.7 mm to (157.8, 29.6)
- moved D3 62.2 mm to (137.6, 30.4), turned to 90 degrees
- moved R21 58.4 mm to (154.9, 10.8)
- moved Q6 54.5 mm to (140.9, 24.5), turned to 270 degrees
- moved R22 54.4 mm to (154.2, 13.5), turned to 270 degrees
- moved C17 53.4 mm to (140.9, 21.8)
- moved D5 49.2 mm to (130.7, 21.8), turned to 270 degrees
- moved C12 48.2 mm to (205.2, 31.4)
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Connections:
- C10 pad 2: Net-(C10-Pad2) -> GND
- C11 pad 2: Net-(C10-Pad2) -> GND
- U1 pad 17: Net-(U1-Pad17) -> /CHARGE_EN
- U4 pad 1: Net-(C10-Pad2) -> GND
Routing:
- net Net-(BT1-Pad2): track 24.5 -> 101.6 mm
- net VBUS: track 0.00 -> 40.5 mm, vias 0 -> 4
- net Net-(D5-Pad1): track 0.00 -> 35.5 mm, vias 0 -> 2
- net +BATT: track 83.3 -> 103.0 mm
- net GND: track 13.4 -> 31.2 mm, vias 15 -> 19
- net Net-(C17-Pad1): track 0.00 -> 17.2 mm
- net +3V3: track 25.9 -> 8.94 mm, vias 2 -> 0
- net Net-(Q3-Pad1): track 0.00 -> 12.7 mm, vias 0 -> 2
- net /BATT_SENSE: track 10.8 -> 2.77 mm
- net Net-(Q5-Pad1): track 0.00 -> 7.19 mm
- net Net-(C10-Pad1): track 0.00 -> 6.53 mm
- net Net-(C16-Pad1): track 0.00 -> 5.78 mm
- net /BUTTON: track 0.00 -> 5.47 mm, vias 0 -> 1
- net /CHARGE_EN: track 0.00 -> 5.44 mm, vias 0 -> 1
- net Net-(D4-Pad3): track 0.00 -> 4.27 mm
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- added copper zone on F.Cu, net /+BATT_SWITCH
- added copper zone on F.Cu, net VBUS
- removed copper zone on F.Cu, net +BATT_SW
Other:
- outline, holes or cut-outs redrawn
- board text removed: "PA1"
- board text removed: "PA2"
- board text removed: "PA5"
- board text removed: "PA6"

Commit message: Rev 2
Parts:
- removed BT1: LI_ON, SamacSys_Parts:1043P
- removed J1: GPIO, Connector_PinHeader_2.54mm:PinHeader_1x06_P2.54mm_Vertical
- removed TP1: +BATT_IN, TestPoint:TestPoint_Pad_D1.0mm
- removed TP2: -BATT_IN, TestPoint:TestPoint_Pad_D1.0mm
- removed TP3: 5V_FB, TestPoint:TestPoint_Pad_D1.0mm
- removed TP4: -BATT_OUT, TestPoint:TestPoint_Pad_D1.0mm
- removed TP7: BATT_SENSE, TestPoint:TestPoint_Pad_D1.0mm
- added J6: +BATT, LedGateController:Battery Pad, F.Cu at (2.70, 2.70)
- added J7: -BATT, LedGateController:Battery Pad, F.Cu at (2.70, 22.3)
- moved J2 138.0 mm to (66.5, 2.00), turned to 270 degrees
- moved TP5 138.0 mm to (72.5, 6.50)
- moved R6 137.5 mm to (59.4, 15.0), turned to 270 degrees
- moved TP6 136.4 mm to (76.0, 15.0)
- moved Q4 135.3 mm to (62.1, 15.0)
- moved C12 134.1 mm to (72.9, 9.18)
- moved C14 134.0 mm to (72.9, 11.5)
- moved C13 133.9 mm to (69.4, 18.0)
- moved R12 133.9 mm to (60.2, 17.8), turned to 180 degrees
- moved J3 133.8 mm to (76.8, 17.9)
- moved U5 133.8 mm to (77.0, 11.9)
- moved C6 121.5 mm to (44.6, 20.8), turned to 90 degrees
- moved C4 115.4 mm to (44.3, 13.5), turned to 0 degrees
- moved C3 115.0 mm to (46.6, 20.8)
- moved R15 114.9 mm to (44.3, 11.5)
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Connections:
- net Net-(BT1-Pad2) renamed /-BATT
- J2 pad 4: /SWDIO -> /SWCLK
- J2 pad 5: /SWCLK -> /SWDIO
- J4 pad 4: Net-(J4-Pad4) -> (no net)
- J5 pad 6: Net-(J5-Pad6) -> (no net)
- U1 pad 1: Net-(U1-Pad1) -> (no net)
- U1 pad 10: Net-(U1-Pad10) -> (no net)
- U1 pad 12: /PWR_LATCH -> /LED_DATA_3V3
- U1 pad 13: Net-(U1-Pad13) -> (no net)
- U1 pad 14: /BATT_SENSE -> (no net)
- U1 pad 15: Net-(U1-Pad15) -> (no net)
- U1 pad 16: Net-(U1-Pad16) -> (no net)
- U1 pad 17: /CHARGE_EN -> (no net)
- U1 pad 18: Net-(U1-Pad18) -> /BATT_SENSE
- U1 pad 19: Net-(U1-Pad19) -> (no net)
- U1 pad 2: Net-(U1-Pad2) -> (no net)
- U1 pad 20: Net-(U1-Pad20) -> (no net)
- U1 pad 21: Net-(U1-Pad21) -> (no net)
- U1 pad 22: Net-(U1-Pad22) -> (no net)
- U1 pad 25: Net-(U1-Pad25) -> /BUTTON
- U1 pad 26: Net-(U1-Pad26) -> /PWR_LATCH
- U1 pad 27: Net-(U1-Pad27) -> /CHARGE_PROG_500MA
- U1 pad 28: Net-(U1-Pad28) -> /CHARGE_PROG_1A
- U1 pad 3: Net-(U1-Pad3) -> (no net)
- U1 pad 30: /BUTTON -> /CHARGE_EN
- U1 pad 31: /LED_DATA_3V3 -> (no net)
- U1 pad 38: Net-(U1-Pad38) -> (no net)
- U1 pad 39: Net-(U1-Pad39) -> (no net)
- U1 pad 4: Net-(U1-Pad4) -> (no net)
- U1 pad 40: Net-(U1-Pad40) -> (no net)
- U1 pad 41: Net-(U1-Pad41) -> (no net)
- U1 pad 42: Net-(U1-Pad42) -> (no net)
- U1 pad 43: Net-(U1-Pad43) -> (no net)
- U1 pad 45: Net-(U1-Pad45) -> (no net)
- U1 pad 46: Net-(U1-Pad46) -> (no net)
- U1 pad 5: Net-(U1-Pad5) -> (no net)
- U1 pad 6: Net-(U1-Pad6) -> (no net)
- U2 pad 6: Net-(U2-Pad6) -> (no net)
- U3 pad 4: Net-(U3-Pad4) -> (no net)
Routing:
- net +BATT: track 103.0 -> 13.8 mm
- net /-BATT: track 101.6 -> 14.1 mm
- net +3V3: track 8.94 -> 95.4 mm, vias 0 -> 8
- net /BATT_SENSE: track 2.77 -> 51.0 mm, vias 1 -> 2
- net /CHARGE_EN: track 5.44 -> 53.6 mm, vias 1 -> 2
- net /BUTTON: track 5.47 -> 46.3 mm, vias 1 -> 2
- net /PWR_LATCH: track 1.28 -> 38.8 mm, vias 1 -> 2
- net Net-(J5-Pad2): track 1.44 -> 36.5 mm, vias 1 -> 2
- net /NRST: track 0.00 -> 30.5 mm, vias 0 -> 1
- net /LED_DATA_3V3: track 3.55 -> 28.6 mm, vias 0 -> 2
- net /SWCLK: track 0.00 -> 24.8 mm, vias 0 -> 1
- net /SWDIO: track 0.24 -> 22.0 mm, vias 0 -> 1
- net Net-(JP2-Pad1): track 0.00 -> 20.3 mm, vias 0 -> 2
- net Net-(C13-Pad1): track 0.00 -> 18.6 mm
- net /CHARGE_PROG_1A: track 0.00 -> 16.6 mm, vias 0 -> 2
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Other:
- board size 144.5 x 25 mm -> 80 x 25 mm

Commit message: rev 2 ordered
Parts:
- removed the ? at (184.8, 4.00)
- moved C1 0.90 mm to (57.4, 10.0)
- moved R11 0.90 mm to (58.3, 7.29)
- moved JP2 0.90 mm to (56.1, 7.30)
- renumbered J6 to +
Connections:
- U1 pad 11: /LED_EN -> (no net)
- U1 pad 21: (no net) -> /LED_EN
Routing:
- net /LED_EN: track 5.48 -> 13.5 mm, vias 0 -> 2
- net Net-(JP2-Pad1): track 20.3 -> 25.5 mm
- net /NRST: track 30.5 -> 28.9 mm
- net +3V3: track 95.4 -> 94.8 mm
- net /LED_DATA_5V: track 10.5 -> 11.1 mm, vias 1 -> 0
Other:
- rule pad_to_mask_clearance: 0.0508 -> 0
