File: LedGateController.sch (KiCad schematic (older format))
At the start: 48 parts, among them J1 5050_OUT, J2 SWD, J3 GPIO, Q1 FS8205A, Q2 AO3400A, Q3 AO3400A, Q4 AO3400A, SW1 SW_SPST, SW2 BUTTON, U1 AP2127N-3.3, U2 MT3608, U3 DW01, U4 STM32F030F4Px

Commit message: Move to footprints
Parts:
- removed Q3, Q4: AO3400A, Package_TO_SOT_SMD:SOT-23, symbol MiscParts:AO3400A
- removed R11, R12, R13: 100, Resistor_SMD:R_0805_2012Metric_Pad1.15x1.40mm_HandSolder, symbol Device:R
- removed TP3: +3V3, TestPoint:TestPoint_THTPad_2.0x2.0mm_Drill1.0mm, symbol Connector:TestPoint
- removed TP4: +12V, TestPoint:TestPoint_THTPad_2.0x2.0mm_Drill1.0mm, symbol Connector:TestPoint
- removed TP7: NRST, TestPoint:TestPoint_THTPad_2.0x2.0mm_Drill1.0mm, symbol Connector:TestPoint
- removed U1: AP2127N-3.3, Package_TO_SOT_SMD:SOT-23, symbol Regulator_Linear:AP2127N-3.3
- added C12, C14: 100n, Capacitor_SMD:C_0805_2012Metric_Pad1.15x1.40mm_HandSolder, symbol Device:C
- added C13: 470u, Capacitor_SMD:CP_Elec_10x7.7, symbol Device:CP
- added Q3: AO3401A, Package_TO_SOT_SMD:SOT-23, symbol Transistor_FET:AO3401A
- added R6, R7: 100, Resistor_SMD:R_0805_2012Metric_Pad1.15x1.40mm_HandSolder, symbol Device:R
- added TP5: LED_DATA_3V3, TestPoint:TestPoint_THTPad_D2.0mm_Drill1.0mm, symbol Connector:TestPoint
- added TP6: LED_DATA_5V, TestPoint:TestPoint_THTPad_D2.0mm_Drill1.0mm, symbol Connector:TestPoint
- added U4: XC6206P332MR, Package_TO_SOT_SMD:SOT-23, symbol Regulator_Linear:XC6206PxxxMR
- added U5: PI4ULS5V201, Package_TO_SOT_SMD:SOT-23-6_Handsoldering, symbol MiscParts:PI4ULS5V201
- BT1: value 18650 -> LI_ON; Digikey Part (none) -> https://www.digikey.co.uk/product-detail/en/keystone-electr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
- C1: renamed from C9; value 100nF -> 100n; footprint (none) -> Capacitor_SMD:C_0805_2012Metric_Pad1.15x1.40mm_HandSolder; LCSC Part (none) -> https://lcsc.com/product-detail/Multilayer-Ceramic-Capacito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
- C10: renamed from C1; value 0.1uF -> 1u; LCSC Part (none) -> https://lcsc.com/product-detail/Multilayer-Ceramic-Capacito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
- C11: renamed from C4; value 0.1uF -> 1u; LCSC Part (none) -> https://lcsc.com/product-detail/Multilayer-Ceramic-Capacito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
- C2: value 22uF -> 22u; footprint (none) -> Capacitor_SMD:C_0805_2012Metric_Pad1.15x1.40mm_HandSolder; LCSC Part (none) -> https://lcsc.com/product-detail/Multilayer-Ceramic-Capacito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
- C3: renamed from C6; value 100nF -> 100n; footprint (none) -> Capacitor_SMD:C_0805_2012Metric_Pad1.15x1.40mm_HandSolder; LCSC Part (none) -> https://lcsc.com/product-detail/Multilayer-Ceramic-Capacito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
- C4: renamed from C10; value 100nF -> 100n; footprint (none) -> Capacitor_SMD:C_0805_2012Metric_Pad1.15x1.40mm_HandSolder; LCSC Part (none) -> https://lcsc.com/product-detail/Multilayer-Ceramic-Capacito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
- C5: renamed from C3; value 0.1uF -> 100n; LCSC Part (none) -> https://lcsc.com/product-detail/Multilayer-Ceramic-Capacito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
- C6: renamed from C11; value 4.7uF -> 4u7; footprint (none) -> Capacitor_SMD:C_0805_2012Metric_Pad1.15x1.40mm_HandSolder; LCSC Part (none) -> https://lcsc.com/product-detail/Multilayer-Ceramic-Capacito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
- C7: renamed from C12; value 1uF -> 1u; footprint (none) -> Capacitor_SMD:C_0805_2012Metric_Pad1.15x1.40mm_HandSolder
- C8: renamed from C13; value 10nF -> 10n; footprint (none) -> Capacitor_SMD:C_0805_2012Metric_Pad1.15x1.40mm_HandSolder; LCSC Part (none) -> https://lcsc.com/product-detail/Multilayer-Ceramic-Capacito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
- C9: renamed from C5; value 22uF -> 22u; footprint (none) -> Capacitor_SMD:C_0805_2012Metric_Pad1.15x1.40mm_HandSolder; LCSC Part (none) -> https://lcsc.com/product-detail/Multilayer-Ceramic-Capacito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
- D1: value D_Schottky -> SS22; footprint (none) -> Diode_SMD:D_SMA_Handsoldering; LCSC Part (none) -> https://lcsc.com/product-detail/Schottky-Barrier-Diodes-SBD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
- D2: footprint (none) -> LED_SMD:LED_0805_2012Metric_Pad1.12x1.40mm_HandSolder; LCSC Part (none) -> https://jlcpcb.com/parts/componentSearch?secondSortUuid=ac4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
- J1: renamed from J3; footprint (none) -> Connector_PinHeader_2.54mm:PinHeader_1x10_P2.54mm_Vertical
- J2: footprint (none) -> Connector_PinHeader_2.54mm:PinHeader_1x05_P2.54mm_Vertical; symbol Connector:Conn_01x04_Male -> Connector:Conn_01x05_Male
- J3: renamed from J1; value 5050_OUT -> LED_OUT; footprint (none) -> Connector_PinHeader_2.54mm:PinHeader_1x03_P2.54mm_Horizontal; symbol Connector:Conn_01x04_Male -> Connector:Conn_01x03_Male
- L1: value 22uH -> 22u; footprint (none) -> Inductor_SMD:L_10.4x10.4_H4.8; LCSC Part (none) -> https://lcsc.com/product-detail/Power-Inductors_TDG-TMAX-10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
- Q1: footprint SOP65P640X120-8N -> Package_SO:TSSOP-8_4.4x3mm_P0.65mm; LCSC Part (none) -> https://lcsc.com/product-detail/MOSFET_Fortune-Semicon-FS82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
- Q2: LCSC Part (none) -> https://lcsc.com/product-detail/MOSFET_UMW-Youtai-Semicondu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
- R1: value 100R -> 100; LCSC Part (none) -> https://lcsc.com/product-detail/Chip-Resistor-Surface-Mount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
- R10: renamed from R9; value 33k -> 100K; LCSC Part (none) -> https://lcsc.com/product-detail/Chip-Resistor-Surface-Mount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
- R2: renamed from R6; value 100k -> 100K; LCSC Part (none) -> https://lcsc.com/product-detail/Chip-Resistor-Surface-Mount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
- R3: renamed from R2; value 5.6k -> 15K; LCSC Part (none) -> https://lcsc.com/product-detail/Chip-Resistor-Surface-Mount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
- R4: renamed from R3; value 100k -> 110K; LCSC Part (none) -> https://lcsc.com/product-detail/Chip-Resistor-Surface-Mount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
- R5: renamed from R4; value 1kR -> 1K; LCSC Part (none) -> https://lcsc.com/product-detail/Chip-Resistor-Surface-Mount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
- R8: renamed from R5; value 330R -> 150; LCSC Part (none) -> https://lcsc.com/product-detail/Chip-Resistor-Surface-Mount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
- R9: renamed from R8; value 100k -> 50K; LCSC Part (none) -> https://lcsc.com/product-detail/Chip-Resistor-Surface-Mount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
- SW1: renamed from SW2; footprint (none) -> Button_Switch_THT:SW_PUSH_6mm; LCSC Part (none) -> https://lcsc.com/product-detail/Tactile-Switches_SHOU-HAN-T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
- SW2: renamed from SW1; value SW_SPST -> ON_OFF; footprint (none) -> Button_Switch_THT:SW_CuK_OS102011MA1QN1_SPDT_Angled; symbol Switch:SW_SPST -> Switch:SW_SPDT; LCSC Part (none) -> https://lcsc.com/product-detail/Toggle-Switches_C-K_OS10201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
- TP2: footprint TestPoint:TestPoint_THTPad_2.0x2.0mm_Drill1.0mm -> TestPoint:TestPoint_THTPad_D2.0mm_Drill1.0mm
- TP3: renamed from TP8; value 12V_FB -> 5V_FB; footprint TestPoint:TestPoint_THTPad_2.0x2.0mm_Drill1.0mm -> TestPoint:TestPoint_THTPad_D2.0mm_Drill1.0mm
- U1: renamed from U4; LCSC Part (none) -> https://lcsc.com/product-detail/Others_STMicroelectronics_S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
- U2: footprint SOT95P280X145-6N -> Package_TO_SOT_SMD:SOT-23-6_Handsoldering; LCSC Part (none) -> https://lcsc.com/product-detail/DC-DC-Converters_MT3608_C84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
- U3: footprint SOT95P280X135-6N -> Package_TO_SOT_SMD:SOT-23-6_Handsoldering; LCSC Part (none) -> https://lcsc.com/product-detail/MOSFET_DW01_C181096.html; Manufacturer_Name Slkor -> (none)
- renumbered TP6 to TP4, TP5 to TP7
Connections:
- net labels added: +5V, +BATT_SW, LED_DATA_3V3, LED_DATA_5V, LED_EN, NRST, PA6, PA7
- net labels removed: +12V, -BATT, B, G, PA2, PA9, R
- wire segments 138 -> 177
- no-connect marks 5 -> 4
Other:
- note added: "Battery Switch"
- note added: "LED Logic Shifter"
- note added: "LED Supply (5V)"
- note removed: "LED Supply (12V)"
- moved on the sheet: C1, C10, C11, C2, C3, C4, C5, C6, C7, C8, C9, D1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

Commit message: nearly done
Parts:
- J1: footprint Connector_PinHeader_2.54mm:PinHeader_1x10_P2.54mm_Vertical -> Connector_PinHeader_2.54mm:PinHeader_1x06_P2.54mm_Vertical; symbol Connector_Generic:Conn_01x10 -> Connector_Generic:Conn_01x06
- SW1: footprint Button_Switch_THT:SW_PUSH_6mm -> LedGateController:TS-1009B-04326; LCSC Part https://lcsc.com/product-detail/Tactile-Switches_SHOU-HAN-T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 -> https://lcsc.com/product-detail/Tactile-Switches_XUNPU-TS-1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
- SW2: footprint Button_Switch_THT:SW_CuK_OS102011MA1QN1_SPDT_Angled -> SamacSys_Parts:SK12D07VG4NSPA; LCSC Part https://lcsc.com/product-detail/Toggle-Switches_C-K_OS10201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 -> https://lcsc.com/product-detail/Toggle-Switches_SHOU-HAN-SK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
- TP1, TP2, TP3, TP4, TP5, TP6, TP7: footprint TestPoint:TestPoint_THTPad_D2.0mm_Drill1.0mm -> TestPoint:TestPoint_THTPad_D1.5mm_Drill0.7mm
Connections:
- net labels added: PA1, PA2
- net labels removed: PA10, PA3, PA4, PA7
- wire segments 177 -> 173
- no-connect marks 4 -> 6
Other:
- moved on the sheet: C2, C9, D1, L1, R3, R4, TP3, U2

Commit message: Rev. 1 nearly ready!
Connections:
- net +3V3: now also J1.2 (Pin_2), J2.2 (Pin_2); no longer J1.6 (Pin_6), J2.5 (Pin_5)
- net NRST: now also J2.3 (Pin_3); no longer J2.2 (Pin_2)
- net PA1: now also J1.4 (Pin_4); no longer J1.3 (Pin_3)
- net PA2: now also J1.3 (Pin_3); no longer J1.2 (Pin_2)
- net PA5: now also J1.5 (Pin_5); no longer J1.4 (Pin_4)
- net PA6: now also J1.6 (Pin_6); no longer J1.5 (Pin_5)
- net SWDCLK: now also J2.5 (Pin_5); no longer J2.3 (Pin_3)
Changed lines of the file:
@@
 L power:+3V3 #PWR015
 U 1 1 5F189137
-P 3900 4500
-F 0 "#PWR015" H 3900 4350 50  0001 C CNN
-F 1 "+3V3" H 3769 4652 50  0000 L CNN
-F 2 "" H 3900 4500 50  0001 C CNN
-F 3 "" H 3900 4500 50  0001 C CNN
-	1    3900 4500
-	1    0    0    -1
+P 3900 4850
+F 0 "#PWR015" H 3900 4700 50  0001 C CNN
+F 1 "+3V3" V 3900 4950 50  0000 L CNN
+F 2 "" H 3900 4850 50  0001 C CNN
+F 3 "" H 3900 4850 50  0001 C CNN
+	1    3900 4850
+	0    -1   -1   0
 $EndComp
 Wire Wire Line
@@
 	4300 3500 4300 3550
 Wire Wire Line
-	3900 4550 3900 4500
-Wire Wire Line
 	3900 5000 3900 4950
 Wire Wire Line
@@
 	0    -1   -1   0
 $EndComp
-Text Label 3700 6850 2    50   ~ 0
+Text Label 3700 6950 2    50   ~ 0
 PA1
-Text Label 3700 7050 2    50   ~ 0
+Text Label 3700 7150 2    50   ~ 0
 PA6
 Wire Wire Line
@@
 Wire Wire Line
 	3700 7150 3750 7150
-Text Label 3700 6950 2    50   ~ 0
+Text Label 3700 7050 2    50   ~ 0
 PA5
-Text Label 3700 6750 2    50   ~ 0
+Text Label 3700 6850 2    50   ~ 0
 PA2
 $Comp
@@
 	0    1    1    0
 $EndComp
+NoConn ~ 2650 6800
+NoConn ~ 2650 6900
 $Comp
 L power:+3V3 #PWR011
 U 1 1 5F2CFCAD
-P 3700 7150
-F 0 "#PWR011" H 3700 7000 50  0001 C CNN
-F 1 "+3V3" V 3700 7250 50  0000 L CNN
-F 2 "" H 3700 7150 50  0001 C CNN
-F 3 "" H 3700 7150 50  0001 C CNN
-	1    3700 7150
+P 3700 6750
+F 0 "#PWR011" H 3700 6600 50  0001 C CNN
+F 1 "+3V3" V 3700 6850 50  0000 L CNN
+F 2 "" H 3700 6750 50  0001 C CNN
+F 3 "" H 3700 6750 50  0001 C CNN
+	1    3700 6750
 	0    -1   -1   0
 $EndComp
-NoConn ~ 2650 6800
-NoConn ~ 2650 6900
+Text Label 3900 4750 2    50   ~ 0
+NRST
+Text Label 3900 4550 2    50   ~ 0
+SWDCLK
 Text Label 3900 4650 2    50   ~ 0
 SWDIO
-Text Label 3900 4750 2    50   ~ 0
-SWDCLK
-Text Label 3900 4850 2    50   ~ 0
-NRST
 $EndSCHEMATC

Commit message: Fix inductor schematic
Parts:
- L1: footprint Inductor_SMD:L_10.4x10.4_H4.8 -> LedGateController:YT1040-220M
Changed lines of the file:
@@
 F 0 "L1" V 2040 3700 50  0000 C CNN
 F 1 "22u" V 1949 3700 50  0000 C CNN
-F 2 "Inductor_SMD:L_10.4x10.4_H4.8" H 1850 3700 50  0001 C CNN
+F 2 "LedGateController:YT1040-220M" V 1750 3650 50  0001 C CNN
 F 3 "~" H 1850 3700 50  0001 C CNN
 F 4 "https://lcsc.com/product-detail/Power-Inductors_TDG-TMAX-1040-220-M_C429809.html" V 1850 3700 50  0001 C CNN "LCSC Part"

Commit message: Update schematic
Parts:
- removed Q2: AO3400A, Package_TO_SOT_SMD:SOT-23, symbol MiscParts:AO3400A
- removed SW2: ON_OFF, SamacSys_Parts:SK12D07VG4NSPA, symbol Switch:SW_SPDT
- removed U1: STM32F030F4Px, Package_SO:TSSOP-20_4.4x6.5mm_P0.65mm, symbol MCU_ST_STM32F0:STM32F030F4Px
- added C15: 1u, Capacitor_SMD:C_0805_2012Metric, symbol Device:C
- added C16, C17: 100n, Capacitor_SMD:C_0805_2012Metric, symbol Device:C
- added C18, C19: 4u7, Capacitor_SMD:C_0805_2012Metric, symbol Device:C
- added D3, D4: D_x2_KCom_AAK, Package_TO_SOT_SMD:SOT-23, symbol Device:D_x2_KCom_AAK
- added D5: CHARGE_LED, LED_SMD:LED_0805_2012Metric, symbol Device:LED
- added J4: USB_B_Micro, SamacSys_Parts:U254051T4BHJ25S2S, symbol Connector:USB_B_Micro
- added J5: TP4056, SamacSys_Parts:SOIC127P600X175-9N, symbol SamacSys_Parts:TP4056
- added JP2: BOOT, Jumper:SolderJumper-2_P1.3mm_Open_Pad1.0x1.5mm, symbol Jumper:SolderJumper_2_Open
- added Q2, Q4, Q6: AO3401A, Package_TO_SOT_SMD:SOT-23, symbol Transistor_FET:AO3401A
- added Q5: AO3400A, Package_TO_SOT_SMD:SOT-23, symbol MiscParts:AO3400A
- added R11, R12, R16, R18, R19, R20, R23: 100K, Resistor_SMD:R_0805_2012Metric, symbol Device:R
- added R13, R14: 1K, Resistor_SMD:R_0805_2012Metric, symbol Device:R
- added R15: 1K5, Resistor_SMD:R_0805_2012Metric, symbol Device:R
- added R17: 100, Resistor_SMD:R_0805_2012Metric, symbol Device:R
- added R21, R22: 1.5K, Resistor_SMD:R_0805_2012Metric, symbol Device:R
- added R24: 250, Resistor_SMD:R_0805_2012Metric, symbol Device:R
- added U1: STM32F103C8Tx, Package_QFP:LQFP-48_7x7mm_P0.5mm, symbol MCU_ST_STM32F1:STM32F103C8Tx
- C1, C10, C11, C12, C14, C2, C3, C4, C5, C6, C8, C9: footprint Capacitor_SMD:C_0805_2012Metric_Pad1.15x1.40mm_HandSolder -> Capacitor_SMD:C_0805_2012Metric
- C7: value 1u -> 100n; footprint Capacitor_SMD:C_0805_2012Metric_Pad1.15x1.40mm_HandSolder -> Capacitor_SMD:C_0805_2012Metric; LCSC Part (none) -> https://lcsc.com/product-detail/Multilayer-Ceramic-Capacito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
- D2: value LED -> PWR_LED; footprint LED_SMD:LED_0805_2012Metric_Pad1.12x1.40mm_HandSolder -> LED_SMD:LED_0805_2012Metric
- R1, R3, R4, R5, R6, R9: footprint Resistor_SMD:R_0805_2012Metric_Pad1.15x1.40mm_HandSolder -> Resistor_SMD:R_0805_2012Metric
- R10: value 100K -> 150K; footprint Resistor_SMD:R_0805_2012Metric_Pad1.15x1.40mm_HandSolder -> Resistor_SMD:R_0805_2012Metric
- R2: value 100K -> 100; footprint Resistor_SMD:R_0805_2012Metric_Pad1.15x1.40mm_HandSolder -> Resistor_SMD:R_0805_2012Metric; LCSC Part https://lcsc.com/product-detail/Chip-Resistor-Surface-Mount_Uniroyal-Elec-0805W8F1003T5E_C17407.html/?href=jlc-SMT -> https://lcsc.com/product-detail/Chip-Resistor-Surface-Mount_Uniroyal-Elec-0805W8F1502T5E_C17475.html/?href=jlc-SMT
- R7: value 100 -> 100K; footprint Resistor_SMD:R_0805_2012Metric_Pad1.15x1.40mm_HandSolder -> Resistor_SMD:R_0805_2012Metric; LCSC Part https://lcsc.com/product-detail/Chip-Resistor-Surface-Mount_Uniroyal-Elec-0805W8F1000T5E_C17408.html/?href=jlc-SMT -> https://lcsc.com/product-detail/Chip-Resistor-Surface-Mount_Uniroyal-Elec-0805W8F1502T5E_C17475.html/?href=jlc-SMT
- R8: value 150 -> 250; footprint Resistor_SMD:R_0805_2012Metric_Pad1.15x1.40mm_HandSolder -> Resistor_SMD:R_0805_2012Metric
- TP7: value BATT_ADC -> BATT_SENSE
- U2, U3, U5: footprint Package_TO_SOT_SMD:SOT-23-6_Handsoldering -> Package_TO_SOT_SMD:SOT-23-6
Connections:
- net +3V3: now also C3.1, C15.1, JP2.2 (B), R15.1, U1.24 (VDD), U1.36 (VDD), U1.48 (VDD), U1.9 (VDDA); no longer C7.1
- net +5V: now also D3.1 (A), Q4.2 (S), R12.1; no longer C10.1, C13.1, J3.3 (Pin_3), U4.3 (VI)
- net +BATT: now also SW1.2, C19.1, J5.5 (BAT), R20.1; no longer R7.1
- net BUTTON: now also R13.1, R14.2, U1.30 (PA9)
- net GND: now also C13.2, C7.1, J3.1 (Pin_1), R7.2, C15.2, C16.2, C18.2, C19.2, J4.5 (GND), J5.1 (TEMP1), J5.3 (GND_3), J5.9 (EP), Q5.2 (S), R11.2, R13.2, R16.2, R18.2, R19.2, R23.2, U1.23 (VSS), U1.35 (VSS), U1.47 (VSS), U1.8 (VSSA); no longer C10.2, C11.2, C7.2, R2.2, SW1.2, U4.1 (GND)
- net LED_DATA_3V3: now also U1.31 (PA10)
- net LED_EN: now also U1.11 (PA1)
- net NRST: now also C7.2, U1.7 (NRST); no longer C3.1
- net SWDIO: now also U1.34 (PA13)
- net at R6.2: now also Q4.1 (G), R12.2
- net at Q3.1 (G): now also Q5.3 (D), R20.2
- net at R2.1: now also R7.1, Q2.1 (G)
- net +BATT_SW renamed +BATT_SWITCH
- net +BATT_SWITCH: now also Q2.2 (S); no longer U2.4 (EN)
- net BATT_ADC renamed BATT_SENSE
- net BATT_SENSE: now also U1.14 (PA4)
- net PA1: no longer names the net of J1.4 (Pin_4)
- net PA2: no longer names the net of J1.3 (Pin_3)
- net PA5: no longer names the net of J1.5 (Pin_5)
- net PA6: no longer names the net of J1.6 (Pin_6)
- net SWDCLK renamed SWCLK
- net SWCLK: now also U1.37 (PA14)
- new net: Q2.3 (D), U2.4 (EN)
- new net: C13.1, J3.3 (Pin_3), Q4.3 (D)
- new net: C10.1, D3.3 (K), U4.3 (VI)
- new net: C10.2, C11.2, U4.1 (GND)
- new net: JP2.1 (A), R11.1, U1.44 (BOOT0)
- new net: C17.1, J4.1 (VBUS), Q6.2 (S), R16.1
- new net: C16.1, D4.2 (A), R14.1
- new net: D4.3 (K), R17.2
- new net: Q5.1 (G), R17.1, R18.1
- new net: J5.2 (PROG2), R21.1
- new net: D5.1 (K), J5.7 (~CHRG)
- new net: D5.2 (A), R24.2
- new net: C17.2, Q6.1 (G), R19.1
- new net CHARGE_EN: J5.8 (CE), R23.1
- new net CHARGE_PROG_1A: R21.2, R22.1
- new net CHARGE_PROG_500MA: R22.2
- new net PWR_LATCH: D4.1 (A), U1.12 (PA2)
- new net USBDM: J4.2 (D-), U1.32 (PA11)
- new net USBDP: J4.3 (D+), R15.2, U1.33 (PA12)
- new net VBUS: C18.1, D3.2 (A), J5.4 (VCC4), Q6.3 (D), R2.2, R24.1, U1.29 (PA8)
- no-connect marks 6 -> 32
Other:
- note added: "Battery Input"
- note added: "Regulators"
- note added: "Soft Power + Button"
- note added: "USB Input"
- note removed: "Battery Input (3.7V)"
- note removed: "Battery Switch"
- note removed: "Button"
- note removed: "LED Supply (5V)"
- note removed: "MCU Supply (3.3V)"
- moved on the sheet: C10, C11, C12, C13, C14, C2, C9, D1, D2, J1, J2, J3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

Commit message: Rewire top section
Parts:
- TP1, TP2, TP3, TP4, TP5, TP6, TP7: footprint TestPoint:TestPoint_THTPad_D1.5mm_Drill0.7mm -> TestPoint:TestPoint_Pad_D1.0mm
Connections:
- net CHARGE_EN: now also U1.17 (PA7)
- net GND: now also C10.2, C11.2, U4.1 (GND)
- no-connect marks 32 -> 31
Changed lines of the file:
@@
 F 0 "TP4" H 4750 2150 50  0000 L CNN
 F 1 "-BATT_OUT" H 4600 2250 50  0000 L CNN
-F 2 "TestPoint:TestPoint_THTPad_D1.5mm_Drill0.7mm" H 5000 1900 50  0001 C CNN
+F 2 "TestPoint:TestPoint_Pad_D1.0mm" H 5000 1900 50  0001 C CNN
 F 3 "~" H 5000 1900 50  0001 C CNN
 	1    4800 1900
@@
 F 0 "TP2" V 800 2050 50  0000 C CNN
 F 1 "-BATT_IN" V 700 2100 50  0000 C CNN
-F 2 "TestPoint:TestPoint_THTPad_D1.5mm_Drill0.7mm" H 1100 1900 50  0001 C CNN
+F 2 "TestPoint:TestPoint_Pad_D1.0mm" H 1100 1900 50  0001 C CNN
 F 3 "~" H 1100 1900 50  0001 C CNN
 	1    900  1900
@@
 F 0 "TP1" V 1100 1400 50  0000 C CNN
 F 1 "+BATT_IN" V 1000 1450 50  0000 C CNN
-F 2 "TestPoint:TestPoint_THTPad_D1.5mm_Drill0.7mm" H 1100 1300 50  0001 C CNN
+F 2 "TestPoint:TestPoint_Pad_D1.0mm" H 1100 1300 50  0001 C CNN
 F 3 "~" H 1100 1300 50  0001 C CNN
 	1    900  1300
@@
 F 0 "TP6" H 9525 8725 50  0000 L CNN
 F 1 "LED_DATA_5V" H 9360 8792 50  0000 L CNN
-F 2 "TestPoint:TestPoint_THTPad_D1.5mm_Drill0.7mm" H 9925 8575 50  0001 C CNN
+F 2 "TestPoint:TestPoint_Pad_D1.0mm" H 9925 8575 50  0001 C CNN
 F 3 "~" H 9925 8575 50  0001 C CNN
 	1    9725 8575
@@
 F 0 "TP5" H 8875 8725 50  0000 L CNN
 F 1 "LED_DATA_3V3" H 8696 8796 50  0000 L CNN
-F 2 "TestPoint:TestPoint_THTPad_D1.5mm_Drill0.7mm" H 9025 8575 50  0001 C CNN
+F 2 "TestPoint:TestPoint_Pad_D1.0mm" H 9025 8575 50  0001 C CNN
 F 3 "~" H 9025 8575 50  0001 C CNN
 	1    8825 8575
@@
 F 0 "TP7" H 9875 2450 50  0000 L CNN
 F 1 "BATT_SENSE" H 9675 2525 50  0000 L CNN
-F 2 "TestPoint:TestPoint_THTPad_D1.5mm_Drill0.7mm" H 10125 2250 50  0001 C CNN
+F 2 "TestPoint:TestPoint_Pad_D1.0mm" H 10125 2250 50  0001 C CNN
 F 3 "~" H 10125 2250 50  0001 C CNN
 	1    9925 2250
@@
 F 0 "TP3" V 3829 3838 50  0000 L CNN
 F 1 "5V_FB" V 3925 3850 50  0000 L CNN
-F 2 "TestPoint:TestPoint_THTPad_D1.5mm_Drill0.7mm" H 4075 3650 50  0001 C CNN
+F 2 "TestPoint:TestPoint_Pad_D1.0mm" H 4075 3650 50  0001 C CNN
 F 3 "~" H 4075 3650 50  0001 C CNN
 	1    3875 3650
@@
 NoConn ~ 3025 10075
 NoConn ~ 4325 10075
-NoConn ~ 4325 9275
 NoConn ~ 4325 9175
 NoConn ~ 4325 9075
@@
 U 1 1 5F872D60
 P 5575 6025
-F 0 "R21" H 5725 6050 50  0000 R CNN
+F 0 "R21" H 5775 6050 50  0000 R CNN
 F 1 "1.5K" H 5800 5975 50  0000 R CNN
 F 2 "Resistor_SMD:R_0805_2012Metric" V 5505 6025 50  0001 C CNN
@@
 U 1 1 5F87371D
 P 5575 6375
-F 0 "R22" H 5725 6400 50  0000 R CNN
+F 0 "R22" H 5775 6425 50  0000 R CNN
 F 1 "1.5K" H 5800 6325 50  0000 R CNN
 F 2 "Resistor_SMD:R_0805_2012Metric" V 5505 6375 50  0001 C CNN
@@
 	1    0    0    -1
 $EndComp
+Text Label 4375 9275 0    50   ~ 0
+CHARGE_EN
+Wire Wire Line
+	4325 9275 4375 9275
+$Comp
+L power:GND #PWR039
+U 1 1 5FC6A6A5
+P 2475 5525
+F 0 "#PWR039" H 2475 5275 50  0001 C CNN
+F 1 "GND" H 2475 5375 50  0001 C CNN
+F 2 "" H 2475 5525 50  0001 C CNN
+F 3 "" H 2475 5525 50  0001 C CNN
+	1    2475 5525
+	1    0    0    -1
+$EndComp

Commit message: Rev 2
Parts:
- removed BT1: LI_ON, SamacSys_Parts:1043P, symbol Device:Battery_Cell
- removed J1: GPIO, Connector_PinHeader_2.54mm:PinHeader_1x06_P2.54mm_Vertical, symbol Connector_Generic:Conn_01x06
- removed TP1: +BATT_IN, TestPoint:TestPoint_Pad_D1.0mm, symbol Connector:TestPoint
- removed TP2: -BATT_IN, TestPoint:TestPoint_Pad_D1.0mm, symbol Connector:TestPoint
- removed TP3: 5V_FB, TestPoint:TestPoint_Pad_D1.0mm, symbol Connector:TestPoint
- removed TP4: -BATT_OUT, TestPoint:TestPoint_Pad_D1.0mm, symbol Connector:TestPoint
- removed TP7: BATT_SENSE, TestPoint:TestPoint_Pad_D1.0mm, symbol Connector:TestPoint
- added J6: +BATT, LedGateController:Battery Pad, symbol Connector_Generic:Conn_01x01
- added J7: -BATT, LedGateController:Battery Pad, symbol Connector_Generic:Conn_01x01
Connections:
- net +BATT: now also J6.1 (Pin_1)
- net BATT_SENSE: now also U1.18 (PB0); no longer U1.14 (PA4)
- net BUTTON: now also U1.25 (PB12); no longer U1.30 (PA9)
- net CHARGE_EN: now also U1.30 (PA9); no longer U1.17 (PA7)
- net CHARGE_PROG_1A: now also U1.28 (PB15)
- net CHARGE_PROG_500MA: now also U1.27 (PB14)
- net LED_DATA_3V3: now also U1.12 (PA2); no longer U1.31 (PA10)
- net PWR_LATCH: now also U1.26 (PB13); no longer U1.12 (PA2)
- net SWCLK: now also J2.4 (Pin_4); no longer J2.5 (Pin_5)
- net SWDIO: now also J2.5 (Pin_5); no longer J2.4 (Pin_4)
- net -BATT: now reaches C5.2, JP1.1 (A), Q1.2 (S1_1), Q1.3 (S1_2), U3.6 (VSS)
- net -BATT: now also J7.1 (Pin_1)
- no-connect marks 31 -> 29
Other:
- note removed: "GPIO"
