File: LedGateController.sch (KiCad schematic (older format))
At the start: 71 parts, among them J2 SWD, J3 LED_OUT, J4 USB_B_Micro, J5 TP4056, J6 +BATT, J7 -BATT, Q1 FS8205A, Q2 AO3401A, Q3 AO3401A, Q4 AO3401A, Q5 AO3400A, Q6 AO3401A, SW1 BUTTON, U1 STM32F103C8Tx, U2 MT3608, U3 DW01, U4 XC6206P332MR, U5 PI4ULS5V201

Commit message: rev 2 ordered
Parts:
- D3, D4: LCSC Part (none) -> https://lcsc.com/product-detail/Diodes-General-Purpose_Nexp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
- J4: LCSC (none) -> https://lcsc.com/product-detail/USB-Connectors_XKB-Connecti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
- J5: LCSC Part (none) -> https://lcsc.com/product-detail/PMIC-Battery-Management_TPO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
- R24, R8: value 250 -> 220
- U1: LCSC Part (none) -> https://lcsc.com/product-detail/ST-Microelectronics_STMicro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
Connections:
- net LED_EN: now also U1.21 (PB10); no longer U1.11 (PA1)
Changed lines of the file:
@@
 Wire Wire Line
 	10925 10675 10975 10675
-Text Label 4325 8675 0    50   ~ 0
+Text Label 3025 9575 2    50   ~ 0
 LED_EN
 Text Notes 11075 10225 2    100  ~ 0
@@
 F 2 "Package_TO_SOT_SMD:SOT-23" H 7775 2100 50  0001 C CNN
 F 3 "~" H 7775 2100 50  0001 C CNN
+F 4 "https://lcsc.com/product-detail/Diodes-General-Purpose_Nexperia-BAV74-215_C85396.html" V 7775 2100 50  0001 C CNN "LCSC Part"
 	1    7775 2100
 	0    -1   -1   0
@@
 F 2 "Package_TO_SOT_SMD:SOT-23" H 1750 5150 50  0001 C CNN
 F 3 "~" H 1750 5150 50  0001 C CNN
+F 4 "https://lcsc.com/product-detail/Diodes-General-Purpose_Nexperia-BAV74-215_C85396.html" V 1750 5150 50  0001 C CNN "LCSC Part"
 	1    1750 5150
 	0    -1   -1   0
@@
 P 7250 5275
 F 0 "R24" V 7425 5325 50  0000 R CNN
-F 1 "250" V 7350 5350 50  0000 R CNN
+F 1 "220" V 7350 5350 50  0000 R CNN
 F 2 "Resistor_SMD:R_0805_2012Metric" V 7180 5275 50  0001 C CNN
 F 3 "~" H 7250 5275 50  0001 C CNN
@@
 F 10 "" H 6925 5075 50  0001 L CNN "Mouser Part Number"
 F 11 "" H 6925 4975 50  0001 L CNN "Mouser Price/Stock"
+F 12 "https://lcsc.com/product-detail/PMIC-Battery-Management_TPOWER-TP4056_C382139.html" H 5675 5775 50  0001 C CNN "LCSC Part"
 	1    5675 5775
 	1    0    0    1
@@
 P 9225 2050
 F 0 "R8" H 9375 2100 50  0000 R CNN
-F 1 "250" H 9425 2025 50  0000 R CNN
+F 1 "220" H 9425 2025 50  0000 R CNN
 F 2 "Resistor_SMD:R_0805_2012Metric" V 9155 2050 50  0001 C CNN
 F 3 "~" H 9225 2050 50  0001 C CNN
@@
 F 2 "SamacSys_Parts:U254051T4BHJ25S2S" H 7225 3775 50  0001 C CNN
 F 3 "~" H 7225 3775 50  0001 C CNN
+F 4 "https://lcsc.com/product-detail/USB-Connectors_XKB-Connectivity-U254-051T-4BHJ25-F2S_C381143.html" H 7075 3825 50  0001 C CNN "LCSC"
 	1    7075 3825
 	1    0    0    -1
@@
 NoConn ~ 3025 8775
 NoConn ~ 3025 9675
-NoConn ~ 3025 9575
 NoConn ~ 3025 8675
 NoConn ~ 4325 9175
@@
 F 2 "Package_QFP:LQFP-48_7x7mm_P0.5mm" H 3125 7375 50  0001 R CNN
 F 3 "http://www.st.com/st-web-ui/static/active/en/resource/technical/document/datasheet/CD00161566.pdf" H 3725 8775 50  0001 C CNN
+F 4 "https://lcsc.com/product-detail/ST-Microelectronics_STMicroelectronics-STM32F103C8T6_C8734.html" H 3725 8775 50  0001 C CNN "LCSC Part"
 	1    3725 8775
 	1    0    0    -1
@@
 Wire Wire Line
 	9650 2250 9975 2250
+NoConn ~ 4325 8675
 $EndSCHEMATC
